Commit message: adjusted frames to match realsense and lidar in rviz

File: ros2_ws/src/go2w_description/urdf/go2w_description_wr.urdf (robot description, URDF)
Before this commit: robot go2w_description, 35 links, 34 joints
Joints:
- joint realsense_joint: origin xyz=0.32 0 0.1 rpy=0 0.05 0 -> xyz=0.34 0 0.12 rpy=0 0 0
