Commit message: preparations for next live robot test

File: ros2_ws/src/go2w_description/urdf/go2w_description_wr3_realsense_frames.urdf (robot description, URDF)
Before this commit: robot go2w_description, 40 links, 39 joints
Links:
- removed link base_link
- removed link front_realsense_base
- removed link front_realsense_body
- removed link front_realsense_flange_left
- removed link front_realsense_flange_right
- removed link front_realsense_mount
- removed link front_realsense_tilt_axis
- added link base, mass 6.921; collision box size=0.3762 0.0935 0.114; visual mesh filename=package://go2w_description/dae/base.dae
- added link rs_base, mass 0; visual mesh filename=package://go2w_description/dae/rs_base.stl scale=0.001 0.001 0.001
- added link rs_d456_solid, mass 0; visual mesh filename=package://go2w_description/dae/rs_D456_Solid.STL scale=0.001 0.001 0.001
- added link rs_flange_left, mass 0; visual mesh filename=package://go2w_description/dae/rs_flange_mirror.stl scale=0.001 0.001 0.001
- added link rs_flange_right, mass 0; visual mesh filename=package://go2w_description/dae/rs_flange.stl scale=0.001 0.001 0.001
- added link rs_mount, mass 0; visual mesh filename=package://go2w_description/dae/rs_mount.stl scale=0.001 0.001 0.001
- added link rs_tilt_axis, mass 0
Joints:
- removed joint front_realsense_base_joint
- removed joint front_realsense_body_joint
- removed joint front_realsense_flange_left_joint
- removed joint front_realsense_flange_right_joint
- removed joint front_realsense_pitch_joint
- removed joint front_realsense_tilt_axis_joint
- added joint rs_base_joint: type fixed, parent base, child rs_base, origin xyz=0.295 0 0.075 rpy=0 0 0, axis 0 0 0
- added joint rs_d456_solid_joint: type fixed, parent rs_mount, child rs_d456_solid, origin xyz=0.02 0 0 rpy=0 0 0, axis 0 0 0
- added joint rs_flange_left_joint: type fixed, parent rs_tilt_axis, child rs_flange_left, origin xyz=0 0.02 -0.028 rpy=0 0 0, axis 0 0 0
- added joint rs_flange_right_joint: type fixed, parent rs_tilt_axis, child rs_flange_right, origin xyz=0 -0.02 -0.028 rpy=0 0 0, axis 0 0 0
- added joint rs_mount_pitch_joint: type fixed, parent rs_tilt_axis, child rs_mount, origin xyz=0 0 0 rpy=0 0 0, axis 0 1 0
- added joint rs_tilt_axis_joint: type fixed, parent rs_base, child rs_tilt_axis, origin xyz=0.005 0 0.032 rpy=0 0 0, axis 0 0 0
- joint FL_hip_joint: parent base_link -> base
- joint FR_hip_joint: parent base_link -> base
- joint Head_upper_joint: parent base_link -> base
- joint RL_hip_joint: parent base_link -> base
- joint RR_hip_joint: parent base_link -> base
- joint front_realsense_sensor_joint: parent front_realsense_body -> rs_d456_solid
- joint imu_joint: parent base_link -> base
- joint radar_joint: parent base_link -> base
